Commit message: Adds launch configs and working urdf joint states

File: ros2_ws/src/wheatley/urdf/bot.xacro (robot description, xacro)
@@ -14,5 +14,5 @@
       <origin xyz="0.0000000000e+00 0.0000000000e+00 0.0000000000e+00" rpy="0.0 0.0 0.0" />
       <geometry>
-        <mesh filename="file://$(find ${package_name})/meshes/base.stl"
+        <mesh filename="package://${package_name}/meshes/base.stl"
           scale="0.001 0.001 0.001" />
       </geometry>
@@ -22,5 +22,5 @@
       <origin xyz="0.0000000000e+00 0.0000000000e+00 0.0000000000e+00" rpy="0.0 0.0 0.0" />
       <geometry>
-        <mesh filename="file://$(find ${package_name})/meshes/base_collision.stl"
+        <mesh filename="package://${package_name}/meshes/base_collision.stl"
           scale="0.001 0.001 0.001" />
       </geometry>
@@ -37,5 +37,5 @@
       <origin xyz="0.0000000000e+00 0.0000000000e+00 -5.0000000000e-02" rpy="0.0 0.0 0.0" />
       <geometry>
-        <mesh filename="file://$(find ${package_name})/meshes/arm.stl" scale="0.001 0.001 0.001" />
+        <mesh filename="package://${package_name}/meshes/arm.stl" scale="0.001 0.001 0.001" />
       </geometry>
       <material name="default_material" />
@@ -44,5 +44,5 @@
       <origin xyz="0.0000000000e+00 0.0000000000e+00 -5.0000000000e-02" rpy="0.0 0.0 0.0" />
       <geometry>
-        <mesh filename="file://$(find ${package_name})/meshes/arm_collision.stl"
+        <mesh filename="package://${package_name}/meshes/arm_collision.stl"
           scale="0.001 0.001 0.001" />
       </geometry>
@@ -68,5 +68,5 @@
       <origin xyz="0.0000000000e+00 1.0000000000e-01 -2.6000000000e-01" rpy="0.0 0.0 0.0" />
       <geometry>
-        <mesh filename="file://$(find ${package_name})/meshes/spinner.stl"
+        <mesh filename="package://${package_name}/meshes/spinner.stl"
           scale="0.001 0.001 0.001" />
       </geometry>
@@ -76,5 +76,5 @@
       <origin xyz="0.0000000000e+00 1.0000000000e-01 -2.6000000000e-01" rpy="0.0 0.0 0.0" />
       <geometry>
-        <mesh filename="file://$(find ${package_name})/meshes/spinner_collision.stl"
+        <mesh filename="package://${package_name}/meshes/spinner_collision.stl"
           scale="0.001 0.001 0.001" />
       </geometry>

File: ros2_ws/src/wheatley/urdf/materials.xacro (robot description, xacro)
@@ -4,4 +4,10 @@
     <color rgba="0.5 0.5 0.5 1.0" />
   </material>
+  <material name="arm_material">
+    <color rgba="0.8 0.2 0.2 1.0" />
+  </material>
+  <material name="spinner_material">
+    <color rgba="0.2 0.8 0.2 1.0" />
+  </material>
   <xacro:property name="existing_contact_coefficients" value="[]" />
 </robot>
